Commit message: fix(sim): model the EPAL 6 as it is built, openings open to the floor
The pallet was eleven boxes: a slab, nine blocks, a slab. Measuring an
800x600 STEP model and the osrf/gazebo_models euro pallet mesh shows the
real thing is twenty two: three bottom boards, nine blocks, three
stringers and seven top boards. Both sources agree and both reproduce
the official EPAL 6 sheet, which states thirteen boards and nine blocks
and dimensions the top-board layout as 217 and 333 mm.

The blocks across the approach face are 100, 145 and 100 mm, not the
uniform 80 mm read off the drawing earlier. That reading was wrong: the
side view draws the bottom boards in front of the blocks, so only a
sliver of each block is visible. Openings are therefore 227.5 mm at
372.5 mm centres, and the prior moves with them. The forks still enter,
with 45 mm of inner and 127.5 mm of outer margin instead of 77.5 and
147.5, and still without raising the mast.

The structural change that matters is underneath. Bottom boards run
under the block columns, so nothing spans beneath a fork opening and a
camera looking in sees the floor. The old continuous slab put a surface
there that no real pallet has.

That surface is exactly what the previous commit taught the detector to
count. Ray-tracing the real assembly gives 286 points in the deck band
at 2 m but 70 at 3 m and 29 at 4 m, against a threshold of 100, so the
lower deck evidence starves again past roughly 2.5 m. Recorded in the
design note with the measurement and three candidate directions, none of
them chosen. The fix is not withdrawn: it stands for the synthetic
catalogue it was measured on, and the v1 replay still reproduces all
hundred stored observations.

Host regression: 759 passed, 1 deselected. Ruff clean.

Co-Authored-By: Claude Opus 5 (1M context) <noreply@anthropic.com>
Claude-Session: https://claude.ai/code/session_01EDwbqCR7d7ymZ6Gm99cASC

File: sim/models/epal6_pallet/pallet.urdf (robot description, URDF)
Before this commit: robot epal6_pallet, 1 links, 0 joints
Links:
- link pallet: geometry collision box size=0.145 0.1 0.078; collision box size=0.145 0.1 0.078
