Commit message: sim+tools+tests+config: EPAL 6 fork spacing 0.3725 m on the measured model (plan S0a) -- dls08_measured fork_spacing_m 0.29 -> 0.3725 (blade centres |y| 0.145 -> 0.18625, nominal blade-to-block 86.25 mm both sides; a hand-adjusted test setting inside the measured range), URDF/MJCF/manifest regenerated, the provisional model untouched; tools/gate_measure.py takes the blade sample points from the URDF the run used (hash-checked; the blade box starts at its root 0.93 m, not the carriage face 0.944 m of the former constants, so e_w is not the 2026-10-08 definition and the points go into each row); sim/isaac/run_pocket_insertion.py hands the model's blade centre and width to the controller (the provisional blades equal its defaults); the N11a/N11b/N14a/N14b bars follow the blade to lateral 0.18625; the historical protection-prediction tests read the pinned 0.29 m URDF, bounds and drive terms (tests/fixtures/near_protection_prediction, byte-identical to b8a5147) and a new test runs the same seed 6 case with the current forks (margin_phys -17.6 -> +21.1 mm, geometry only); comments mark the 0.29 m-measured gaps and withdrawal coefficients, synthetic 0.29 m blade copies are annotated, the model README carries the new provenance row and measurement requests. Not yet valid for Isaac runs: the base scene (S1), the near-field bounds (S2) and the drive terms (S3) are bound to the old URDF and are re-measured next. Local: the 16 affected test files pass (538 tests); the ws1 full suite waits for the node (draining for an admin GPU passthrough teardown). Codex review: no P1/P2, two P3 fixed
Co-Authored-By: Claude Opus 5.5 (1M context) <noreply@anthropic.com>

File: sim/models/dls08_measured/forklift.urdf (robot description, URDF)
Before this commit: robot dls08_measured, 10 links, 9 joints
Joints:
- joint left_fork_tip_fixed: origin xyz=0.95 0.145 0.04 rpy=0 0 0 -> xyz=0.95 0.18625 0.04 rpy=0 0 0
- joint right_fork_tip_fixed: origin xyz=0.95 -0.145 0.04 rpy=0 0 0 -> xyz=0.95 -0.18625 0.04 rpy=0 0 0

Commit message: model+tools+tests: the measured model's fork-tip frame links carry an explicit 0.1 g inertial (assumptions.site_link_mass_kg / site_link_inertia_kgm2, optional keys) -- a URDF link without one became a PhysX body with the default 1 kg, about 2 kg at the fork tips (tyre contact totals 254 N vs 235.4 N); the provisional model has no such key and its output is unchanged; the MJCF is unchanged (sites). Regenerated dls08_measured/forklift.urdf and its manifest. Needs a new base scene (S1) before any Isaac run on it
Co-Authored-By: Claude Opus 5.5 (1M context) <noreply@anthropic.com>

File: sim/models/dls08_measured/forklift.urdf (robot description, URDF)
Before this commit: robot dls08_measured, 10 links, 9 joints
Links:
- link left_fork_tip: mass None -> 0.0001
- link right_fork_tip: mass None -> 0.0001
